File: kicad-template.kicad_pcb (KiCad board)
At the start: 2 copper layers, 0 parts

Commit message: feat: renamed sym,fp libs & added example sch, pcb
Parts:
- added C1: M8-male-straight-4pin_TE_T4040034041-000, kicad-library:Conn_M8_male_straight_4pin_TE_T4040034041-000, F.Cu at (81.2, 45.0)
- added D1: green, LED_SMD:LED_0603_1608Metric_Pad1.05x0.95mm_HandSolder, F.Cu at (69.0, 47.0)
- added G***: LOGO, kicad-library:KF-Logo_2.7x2.2, F.Cu at (65.0, 36.8)
- added R1: 220, Resistor_SMD:R_0603_1608Metric_Pad0.98x0.95mm_HandSolder, F.Cu at (69.0, 43.0)
Routing:
- net Net-(C1-Pad1): track 0.00 -> 12.3 mm
- net GND: track 0.00 -> 12.2 mm
- net Net-(D1-Pad2): track 0.00 -> 2.21 mm
- added copper zone on B.Cu, net GND
- added copper zone on F.Cu, net GND
Other:
- board outline added: 30 x 25 mm
- board text added: "${version}"
- board text added: "kicad-template"
