File: kicad-template.kicad_sch (KiCad schematic)
At the start: 0 parts

Commit message: feat: renamed sym,fp libs & added example sch, pcb
Parts:
- added C1: M8-male-straight-4pin_TE_T4040034041-000, kicad-library:Conn_M8_male_straight_4pin_TE_T4040034041-000, symbol kicad-library-connectors:M8-male-straight-4pin_TE_T4040034041-000
- added D1: green, LED_SMD:LED_0603_1608Metric_Pad1.05x0.95mm_HandSolder, symbol Device:LED_Small
- added R1: 220, Resistor_SMD:R_0603_1608Metric_Pad0.98x0.95mm_HandSolder, symbol Device:R_Small
Connections:
- new net: C1.1, R1.1
- new net: D1.2 (A), R1.2
- new net GND: C1.3, C1.5 (Case), D1.1 (K)
- no-connect marks 0 -> 2
Other:
- note added: "Example LED w/ custom Connector"
Changed lines of the file:
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@@
     (comment 3 "${author}")
+  )
+  (junction (at 43.18 34.29) (diameter 0) (color 0 0 0 0)
+  )
+  (junction (at 43.18 44.45) (diameter 0) (color 0 0 0 0)
+  )
+  (no_connect (at 57.15 38.1))
+  (no_connect (at 57.15 40.64))
+  (polyline (pts (xy 20.32 60.96) (xy 114.3 60.96))
+    (stroke (width 0) (type default) (color 0 0 0 0))
+  )
+  (polyline (pts (xy 20.32 22.86) (xy 20.32 60.96))
+    (stroke (width 0) (type default) (color 0 0 0 0))
+  )
+  (polyline (pts (xy 114.3 22.86) (xy 114.3 60.96))
+    (stroke (width 0) (type default) (color 0 0 0 0))
+  )
+  (wire (pts (xy 43.18 44.45) (xy 43.18 46.99))
+    (stroke (width 0) (type default) (color 0 0 0 0))
+  )
+  (wire (pts (xy 43.18 34.29) (xy 57.15 34.29))
+    (stroke (width 0) (type default) (color 0 0 0 0))
+  )
+  (wire (pts (xy 73.66 35.56) (xy 73.66 34.29))
+    (stroke (width 0) (type default) (color 0 0 0 0))
+  )
+  (wire (pts (xy 43.18 44.45) (xy 57.15 44.45))
+    (stroke (width 0) (type default) (color 0 0 0 0))
+  )
+  (wire (pts (xy 40.64 34.29) (xy 43.18 34.29))
+    (stroke (width 0) (type default) (color 0 0 0 0))
+  )
+  (wire (pts (xy 40.64 44.45) (xy 43.18 44.45))
+    (stroke (width 0) (type default) (color 0 0 0 0))
+  )
+  (polyline (pts (xy 114.3 22.86) (xy 20.32 22.86))
+    (stroke (width 0) (type default) (color 0 0 0 0))
+  )
+  (wire (pts (xy 73.66 34.29) (xy 72.39 34.29))
+    (stroke (width 0) (type default) (color 0 0 0 0))
+  )
+  (text "Example LED w/ custom Connector" (at 20.32 22.86 0)
+    (effects (font (size 1.27 1.27) (thickness 0.254) bold) (justify left bottom))
+  )
+  (symbol (lib_id "kicad-library-connectors:M8-male-straight-4pin_TE_T4040034041-000") (at 59.69 34.29 0) (unit 1)
+    (in_bom yes) (on_board yes)
+    (property "Reference" "C1" (id 0) (at 60.96 27.94 0))
+    (property "Value" "M8-male-straight-4pin_TE_T4040034041-000" (id 1) (at 82.55 30.48 0))
+    (property "Footprint" "kicad-library:Conn_M8_male_straight_4pin_TE_T4040034041-000" (id 2) (at 60.96 60.96 0)
+      (effects (font (size 1.27 1.27)) hide)
+    )
+    (property "Datasheet" "https://www.te.com/commerce/DocumentDelivery/DDEController?Action=srchrtrv&DocNm=T40400340X1000&DocType=Customer+Drawing&DocLang=English" (id 3) (at 62.23 55.88 0)
+      (effects (font (size 1.27 1.27)) hide)
+    )
+    (property "Manufacturer_URL" "https://www.te.com/deu-de/product-T4040034041-000.html" (id 4) (at 59.69 53.34 0)
+      (effects (font (size 1.27 1.27)) hide)
+    )
+    (property "Part-Nr-Digikey" "A126810-ND" (id 5) (at 59.69 58.42 0)
+      (effects (font (size 1.27 1.27)) hide)
+    )
+    (pin "1")
+    (pin "2")
+    (pin "3")
+    (pin "4")
+    (pin "5")
+  )
+  (symbol (lib_id "power:PWR_FLAG") (at 40.64 34.29 90) (unit 1)
+    (in_bom yes) (on_board yes) (fields_autoplaced)
+    (property "Reference" "#FLG01" (id 0) (at 38.735 34.29 0)
+      (effects (font (size 1.27 1.27)) hide)
+    )
+    (property "Value" "PWR_FLAG" (id 1) (at 36.83 34.2899 90)
+      (effects (font (size 1.27 1.27)) (justify left))
+    )
+    (property "Footprint" "" (id 2) (at 40.64 34.29 0)
+      (effects (font (size 1.27 1.27)) hide)
+    )
+    (property "Datasheet" "~" (id 3) (at 40.64 34.29 0)
+      (effects (font (size 1.27 1.27)) hide)
+    )
+    (pin "1")
+  )
+  (symbol (lib_id "Device:LED_Small") (at 43.18 41.91 90) (unit 1)
+    (in_bom yes) (on_board yes)
+    (property "Reference" "D1" (id 0) (at 45.72 40.64 90))
+    (property "Value" "green" (id 1) (at 46.99 43.18 90))
+    (property "Footprint" "LED_SMD:LED_0603_1608Metric_Pad1.05x0.95mm_HandSolder" (id 2) (at 43.18 41.91 90)
+      (effects (font (size 1.27 1.27)) hide)
+    )
+    (property "Datasheet" "~" (id 3) (at 43.18 41.91 90)
+      (effects (font (size 1.27 1.27)) hide)
+    )
+    (pin "1")
+    (pin "2")
+  )
+  (symbol (lib_id "power:GND") (at 43.18 46.99 0) (unit 1)
+    (in_bom yes) (on_board yes) (fields_autoplaced)
+    (property "Reference" "#PWR01" (id 0) (at 43.18 53.34 0)
+      (effects (font (size 1.27 1.27)) hide)
+    )
+    (property "Value" "GND" (id 1) (at 43.18 52.07 0))
+    (property "Footprint" "" (id 2) (at 43.18 46.99 0)
+      (effects (font (size 1.27 1.27)) hide)
+    )
+    (property "Datasheet" "" (id 3) (at 43.18 46.99 0)
+      (effects (font (size 1.27 1.27)) hide)
+    )
+    (pin "1")
+  )
+  (symbol (lib_id "power:GND") (at 73.66 35.56 0) (unit 1)
+    (in_bom yes) (on_board yes) (fields_autoplaced)
+    (property "Reference" "#PWR?" (id 0) (at 73.66 41.91 0)
+      (effects (font (size 1.27 1.27)) hide)
+    )
+    (property "Value" "GND" (id 1) (at 73.66 40.64 0))
+    (property "Footprint" "" (id 2) (at 73.66 35.56 0)
+      (effects (font (size 1.27 1.27)) hide)
+    )
+    (property "Datasheet" "" (id 3) (at 73.66 35.56 0)
+      (effects (font (size 1.27 1.27)) hide)
+    )
+    (pin "1")
+  )
+  (symbol (lib_id "power:PWR_FLAG") (at 40.64 44.45 90) (unit 1)
+    (in_bom yes) (on_board yes) (fields_autoplaced)
+    (property "Reference" "#FLG0101" (id 0) (at 38.735 44.45 0)
+      (effects (font (size 1.27 1.27)) hide)
+    )
+    (property "Value" "PWR_FLAG" (id 1) (at 36.83 44.4499 90)
+      (effects (font (size 1.27 1.27)) (justify left))
+    )
+    (property "Footprint" "" (id 2) (at 40.64 44.45 0)
+      (effects (font (size 1.27 1.27)) hide)
+    )
+    (property "Datasheet" "~" (id 3) (at 40.64 44.45 0)
+      (effects (font (size 1.27 1.27)) hide)
+    )
+    (pin "1")
+  )
+  (symbol (lib_id "Device:R_Small") (at 43.18 36.83 0) (unit 1)
+    (in_bom yes) (on_board yes)
+    (property "Reference" "R1" (id 0) (at 44.45 35.56 0)
+      (effects (font (size 1.27 1.27)) (justify left))
+    )
+    (property "Value" "220" (id 1) (at 44.45 38.1 0)
+      (effects (font (size 1.27 1.27)) (justify left))
+    )
+    (property "Footprint" "Resistor_SMD:R_0603_1608Metric_Pad0.98x0.95mm_HandSolder" (id 2) (at 43.18 36.83 0)
+      (effects (font (size 1.27 1.27)) hide)
+    )
+    (property "Datasheet" "~" (id 3) (at 43.18 36.83 0)
+      (effects (font (size 1.27 1.27)) hide)
+    )
+    (pin "1")
+    (pin "2")
   )
   (sheet_instances
     (path "/" (page "1"))
   )
+  (symbol_instances
+    (path "/3285694c-54b2-45d6-a033-691039f254f3"
+      (reference "#FLG01") (unit 1) (value "PWR_FLAG") (footprint "")
+    )
+    (path "/eb5aac37-aed6-4edd-bdde-2503a462aacc"
+      (reference "#FLG0101") (unit 1) (value "PWR_FLAG") (footprint "")
+    )
+    (path "/a5ae156b-0599-4b66-bd0c-6265e71bcf9a"
+      (reference "#PWR01") (unit 1) (value "GND") (footprint "")
+    )
+    (path "/dd673796-7a32-4f1f-b0c5-d2e15bb16cfe"
+      (reference "#PWR?") (unit 1) (value "GND") (footprint "")
+    )
+    (path "/11df0a9a-26d0-409f-990a-49d7323fbb2a"
+      (reference "C1") (unit 1) (value "M8-male-straight-4pin_TE_T4040034041-000") (footprint "kicad-library:Conn_M8_male_straight_4pin_TE_T4040034041-000")
+    )
+    (path "/55e351e3-7efa-4d55-acad-86a345fc5120"
+      (reference "D1") (unit 1) (value "green") (footprint "LED_SMD:LED_0603_1608Metric_Pad1.05x0.95mm_HandSolder")
+    )
+    (path "/edaf969f-353e-44bd-9eea-e5dbfe1f2308"
+      (reference "R1") (unit 1) (value "220") (footprint "Resistor_SMD:R_0603_1608Metric_Pad0.98x0.95mm_HandSolder")
+    )
+  )
 )
